Commit message: mouning pose correction

File: robots/kukas.urdf.xacro (robot description, xacro)
@@ -3,17 +3,17 @@
 		 xmlns:xacro="http://www.ros.org/wiki/xacro">
   <xacro:include filename="$(find agni_description)/calibration/default_cal.xml"/>
-  <xacro:include filename="$(find agni_description)/urdf/frame.urdf.xacro"/>
+  <xacro:include filename="$(find agni_description)/urdf/frame-half.urdf.xacro"/>
   <xacro:include filename="$(find agni_description)/urdf/kuka_lwr_arm.urdf.xacro"/>
   <xacro:include filename="$(find sr_description)/hand/xacro/full_hand_motor.urdf.xacro" />
-  <xacro:frame prefix="kuka" thickness="0.09" width="1.92" depth="1.82"
-					height="1.26" tableHeight="1.00"/>
+  <xacro:frame-half prefix="kuka" thickness="0.09" width="1.92" depth="1.82"
+						  height="1.26" tableHeight="1.00"/>
   <!-- KUKA arms -->
   <xacro:kuka_lwr_arm parent="kuka_frame" name="left"
-							 right="-1" tool_name="_angle">
+							 right="-1" tool_name="">
 	 <origin xyz="${cal_left_arm_x} ${cal_left_arm_y} ${cal_left_arm_z}"
 				rpy="${cal_left_arm_roll} ${cal_left_arm_pitch} ${cal_left_arm_yaw}"/>
   </xacro:kuka_lwr_arm>
   <xacro:kuka_lwr_arm parent="kuka_frame" name="right"
-							 right="+1" tool_name="_angle">
+							 right="+1" tool_name="">
 	 <origin xyz="${cal_right_arm_x} ${cal_right_arm_y} ${cal_right_arm_z}"
 				rpy="${cal_right_arm_roll} ${cal_right_arm_pitch} ${cal_right_arm_yaw}"/>

File: urdf/frame-half.urdf.xacro (robot description, xacro)
@@ -10,5 +10,5 @@
 	 </visual>
 </xacro:macro>
-<xacro:macro name="frame" params="prefix thickness width depth height tableHeight">
+<xacro:macro name="frame-half" params="prefix thickness width depth height tableHeight">
   <link name="${prefix}_frame">
 	 <!-- horizontal front bar-->
@@ -20,8 +20,4 @@
 		<origin xyz="0 ${depth+thickness/2} ${-thickness/2}" rpy="0 ${-M_PI/2} 0"/>
 	 </xacro:bar>
-	 <!-- horizontal front bar top -->
-	 <xacro:bar thickness="${thickness}" len="${width}">
-		<origin xyz="0 ${-thickness/2} ${height+thickness/2}" rpy="0 ${-M_PI/2} 0"/>
-	 </xacro:bar>
 	 <!-- horizontal rear bar top -->
 	 <xacro:bar thickness="${thickness}" len="${width}">
@@ -29,10 +25,10 @@
 	 </xacro:bar>
 	 <!-- left front pole -->
-	 <xacro:bar thickness="${thickness}" len="${height+2*thickness+tableHeight}">
-		<origin xyz="${-(width+thickness)/2} ${-thickness/2} ${(height-tableHeight)/2}"/>
+	 <xacro:bar thickness="${thickness}" len="${thickness+tableHeight}">
+		<origin xyz="${-(width+thickness)/2} ${-thickness/2} ${-(thickness+tableHeight)/2}"/>
 	 </xacro:bar>
 	 <!-- right front pole -->
-	 <xacro:bar thickness="${thickness}" len="${height+2*thickness+tableHeight}">
-		<origin xyz="${+(width+thickness)/2} ${-thickness/2} ${(height-tableHeight)/2}"/>
+	 <xacro:bar thickness="${thickness}" len="${thickness+tableHeight}">
+		<origin xyz="${+(width+thickness)/2} ${-thickness/2} ${-(thickness+tableHeight)/2}"/>
 	 </xacro:bar>
 	 <!-- left rear pole -->
@@ -54,14 +50,4 @@
 				  rpy="${-M_PI/2} 0 0"/>
 	 </xacro:bar>
-	 <!-- left side top -->
-	 <xacro:bar thickness="${thickness}" len="${depth}">
-		<origin xyz="${-(width+thickness)/2} ${depth/2} ${height+thickness/2}"
-				  rpy="${-M_PI/2} 0 0"/>
-	 </xacro:bar>
-	 <!-- right side top -->
-	 <xacro:bar thickness="${thickness}" len="${depth}">
-		<origin xyz="${+(width+thickness)/2} ${depth/2} ${height+thickness/2}"
-				  rpy="${-M_PI/2} 0 0"/>
-	 </xacro:bar>
   </link>
 </xacro:macro>

File: urdf/kuka_lwr_arm.urdf.xacro (robot description, xacro)
@@ -345,6 +345,8 @@
     </transmission>
     <joint name="${name}_arm_hand_fixed_joint" type="fixed">
+<!--
       <origin xyz="${-right * 0.075} -0.075 -0.094"
               rpy="${0.5*right*M_PI} 0 ${(1.5 + 0.25*right)*M_PI}"/>
+-->
       <parent link="${name}_arm_7_link"/>
       <child link="${name}_arm_hand_link"/>

Commit message: mounting setup for kukas
removed parent from kuka description -> allows to freely position arm
splitted scene description into three parts: frame, right+left arm

File: robots/kukas.urdf.xacro (robot description, xacro)
@@ -6,29 +6,23 @@
   <xacro:include filename="$(find agni_description)/urdf/kuka_lwr_arm.urdf.xacro"/>
   <xacro:include filename="$(find sr_description)/hand/xacro/full_hand_motor.urdf.xacro" />
+<!--
   <xacro:frame-half prefix="kuka" thickness="0.09" width="1.92" depth="1.82"
 						  height="1.26" tableHeight="1.00"/>
+-->
   <!-- KUKA arms -->
-  <xacro:kuka_lwr_arm parent="kuka_frame" name="left"
-							 right="-1" tool_name="">
+  <xacro:kuka_lwr_arm name="right" right="+1" tool_name=""/>
+  <joint name="kuka_right_arm_base_joint" type="fixed">
+	 <origin xyz="${cal_right_arm_x} ${cal_right_arm_y} ${cal_right_arm_z}"
+				rpy="${cal_right_arm_roll} ${cal_right_arm_pitch} ${cal_right_arm_yaw}"/>
+	 <parent link="kuka_frame"/>
+	 <child link="calib_right_arm_base_link"/>
+  </joint>
+  <xacro:kuka_lwr_arm name="left" right="-1" tool_name=""/>
+  <joint name="kuka_left_arm_base_joint" type="fixed">
 	 <origin xyz="${cal_left_arm_x} ${cal_left_arm_y} ${cal_left_arm_z}"
 				rpy="${cal_left_arm_roll} ${cal_left_arm_pitch} ${cal_left_arm_yaw}"/>
-  </xacro:kuka_lwr_arm>
-  <xacro:kuka_lwr_arm parent="kuka_frame" name="right"
-							 right="+1" tool_name="">
-	 <origin xyz="${cal_right_arm_x} ${cal_right_arm_y} ${cal_right_arm_z}"
-				rpy="${cal_right_arm_roll} ${cal_right_arm_pitch} ${cal_right_arm_yaw}"/>
-  </xacro:kuka_lwr_arm>
-<!--
-  <xacro:kuka_lwr_arm parent="kuka_frame" name="left2"
-							 right="-1" tool_name="_angle">
-	 <origin xyz="${cal_base_to_left_arm_x} ${cal_base_to_left_arm_y} ${cal_base_to_left_arm_z}"
-				rpy="${cal_base_to_left_arm_roll} ${cal_base_to_left_arm_pitch} ${cal_base_to_left_arm_yaw}"/>
-  </xacro:kuka_lwr_arm>
-  <xacro:kuka_lwr_arm parent="kuka_frame" name="right2"
-							 right="+1" tool_name="_angle">
-	 <origin xyz="${cal_base_to_right_arm_x} ${cal_base_to_right_arm_y} ${cal_base_to_right_arm_z}"
-				rpy="${cal_base_to_right_arm_roll} ${cal_base_to_right_arm_pitch} ${cal_base_to_right_arm_yaw}"/>
-  </xacro:kuka_lwr_arm>
--->
+	 <parent link="kuka_frame"/>
+	 <child link="calib_left_arm_base_link"/>
+  </joint>
   <!-- Shadow Hands -->
 <!--
@@ -46,19 +40,3 @@
   </joint>
   <xacro:shadowhand_motor/>
-  <transmission name="arm0">
-	 <type>transmission_interface/SimpleTransmission</type>
-	 <joint name="right_arm_0_joint"/>
-	 <actuator name="arm0">
-		<hardwareInterface>EffortJointInterface</hardwareInterface>
-		<mechanicalReduction>1</mechanicalReduction>
-	 </actuator>
-  </transmission>
-  <transmission name="arm0">
-	 <type>transmission_interface/SimpleTransmission</type>
-	 <joint name="left_arm_0_joint"/>
-	 <actuator name="arm0">
-		<hardwareInterface>EffortJointInterface</hardwareInterface>
-		<mechanicalReduction>1</mechanicalReduction>
-	 </actuator>
-  </transmission>
 </robot>

File: urdf/kuka_lwr_arm.urdf.xacro (robot description, xacro)
@@ -1,7 +1,8 @@
 <?xml version="1.0"?>
-<robot xmlns:sensor="http://playerstage.sourceforge.net/gazebo/xmlschema/#sensor"
-       xmlns:controller="http://playerstage.sourceforge.net/gazebo/xmlschema/#controller"
+<robot xmlns:xacro="http://www.ros.org/wiki/xacro"
+		 xmlns:sensor="http://playerstage.sourceforge.net/gazebo/xmlschema/#sensor"
+		 xmlns:controller="http://playerstage.sourceforge.net/gazebo/xmlschema/#controller"
        xmlns:interface="http://playerstage.sourceforge.net/gazebo/xmlschema/#interface">
-  <include filename="$(find agni_description)/urdf/util.urdf.xacro"/>
+  <xacro:include filename="$(find agni_description)/urdf/util.urdf.xacro"/>
   <property name="arm_elem_base_mass" value="2.0"/>
   <property name="arm_elem_link_mass" value="2.0"/>
@@ -13,10 +14,5 @@
   <property name="arm_velocity_scale_factor" value="1"/>
   <!-- right is either 1 (for right arm) or -1 (for left arm) -->
-  <macro name="kuka_lwr_arm" params="parent name right tool_name *origin">
-    <joint name="${parent}_${name}_arm_base_joint" type="fixed">
-      <insert_block name="origin"/>
-      <parent link="${parent}"/>
-      <child link="calib_${name}_arm_base_link"/>
-    </joint>
+  <macro name="kuka_lwr_arm" params="name right tool_name">
     <link name="calib_${name}_arm_base_link">
       <inertial>
