Commit message: worked on urdf files

File: robots/kuka_left.urdf.xacro (robot description, xacro)
@@ -6,7 +6,7 @@
   <xacro:include filename="$(find sr_description)/hand/xacro/full_hand_motor.urdf.xacro" />
   <!-- KUKA arms -->
-  <xacro:kuka_lwr_arm name="left" right="-1" tool_name=""/>
+  <xacro:kuka_lwr_arm name="left_" right="-1" tool_name=""/>
   <joint name="left_arm_hand_mount" type="fixed">
-    <parent link="left_arm_hand_link"/>
+    <parent link="left_arm_hand_mount"/>
     <child link="forearm"/>
     <origin xyz="0 0 0" rpy="0 0 0" />

File: robots/kuka_right.urdf.xacro (robot description, xacro)
@@ -6,8 +6,8 @@
   <xacro:include filename="$(find sr_description)/hand/xacro/full_hand_motor.urdf.xacro" />
   <!-- KUKA arms -->
-  <xacro:kuka_lwr_arm name="right" right="+1" tool_name=""/>
+  <xacro:kuka_lwr_arm name="right_" right="+1" tool_name=""/>
   <!-- Shadow Hands -->
   <joint name="right_arm_hand_mount" type="fixed">
-    <parent link="right_arm_hand_link"/>
+    <parent link="right_arm_hand_mount"/>
     <child link="forearm"/>
     <origin xyz="0 0 0" rpy="0 0 0" />

File: robots/kukas.urdf.xacro (robot description, xacro)
@@ -6,8 +6,6 @@
   <xacro:include filename="$(find agni_description)/urdf/kuka_lwr_arm.urdf.xacro"/>
   <xacro:include filename="$(find sr_description)/hand/xacro/full_hand_motor.urdf.xacro" />
-<!--
   <xacro:frame-half prefix="kuka" thickness="0.09" width="1.92" depth="1.82"
 						  height="1.26" tableHeight="1.00"/>
--->
   <!-- KUKA arms -->
   <xacro:kuka_lwr_arm name="right" right="+1" tool_name=""/>
@@ -26,14 +24,12 @@
   </joint>
   <!-- Shadow Hands -->
-<!--
   <joint name="left_arm_hand_mount" type="fixed">
-    <parent link="left_arm_hand_link"/>
+    <parent link="left_arm_hand_mount"/>
     <child link="forearm"/>
     <origin xyz="0 0 0" rpy="0 0 ${2.35619449}" />
   </joint>
   <xacro:shadowhand_left_motor/>
--->
   <joint name="right_arm_hand_mount" type="fixed">
-    <parent link="right_arm_hand_link"/>
+    <parent link="right_arm_hand_mount"/>
     <child link="forearm"/>
     <origin xyz="0 0 0" rpy="0 0 0" />

File: urdf/kuka_lwr_arm.urdf.xacro (robot description, xacro)
@@ -15,5 +15,5 @@
   <!-- right is either 1 (for right arm) or -1 (for left arm) -->
   <macro name="kuka_lwr_arm" params="name right tool_name">
-    <link name="calib_${name}_arm_base_link">
+    <link name="${name}arm_base_link">
       <inertial>
         <mass value="${arm_elem_base_mass}"/>
@@ -37,8 +37,8 @@
       </collision>
     </link>
-    <gazebo reference="calib_${name}_arm_base_link">
-      <material value="kuka-lwr.material"/>
-    </gazebo>
-    <joint name="${name}_arm_0_joint" type="revolute">
+    <gazebo reference="${name}arm_base_link">
+      <material value="kuka-lwr.material"/>
+    </gazebo>
+    <joint name="${name}arm_0_joint" type="revolute">
       <origin xyz="0 0 0.11" rpy="0 0 0"/>
       <axis xyz="0 0 1"/>
@@ -50,8 +50,13 @@
                          k_velocity="${safety_controller_k_vel}"/>
       <dynamics damping="${joint_damping}"/>
-      <parent link="calib_${name}_arm_base_link"/>
-      <child link="${name}_arm_1_link"/>
-    </joint>
-    <link name="${name}_arm_1_link">
+      <parent link="${name}arm_base_link"/>
+      <child link="${name}arm_1_link"/>
+    </joint>
+    <transmission name="${name}arm_0_trans" type="pr2_mechanism_model/SimpleTransmission">
+      <actuator name="${name}arm_0_motor"/>
+      <joint name="${name}arm_0_joint"/>
+      <mechanicalReduction>1.0</mechanicalReduction>
+    </transmission>
+    <link name="${name}arm_1_link">
       <inertial>
         <mass value="${arm_elem_link_mass}"/>
@@ -74,13 +79,8 @@
       </collision>
     </link>
-    <gazebo reference="${name}_arm_1_link">
-      <material value="kuka-lwr.material"/>
-    </gazebo>
-    <transmission name="${name}_arm_0_trans" type="pr2_mechanism_model/SimpleTransmission">
-      <actuator name="${name}_arm_0_motor"/>
-      <joint name="${name}_arm_0_joint"/>
-      <mechanicalReduction>1.0</mechanicalReduction>
-    </transmission>
-    <joint name="${name}_arm_1_joint" type="revolute">
+    <gazebo reference="${name}arm_1_link">
+      <material value="kuka-lwr.material"/>
+    </gazebo>
+    <joint name="${name}arm_1_joint" type="revolute">
       <origin xyz="0 0 0.20" rpy="0 0 0"/>
       <axis xyz="0 -1 0"/>
@@ -92,8 +92,13 @@
                          k_velocity="${safety_controller_k_vel}"/>
       <dynamics damping="${joint_damping}"/>
-      <parent link="${name}_arm_1_link"/>
-      <child link="${name}_arm_2_link"/>
-    </joint>
-    <link name="${name}_arm_2_link">
+      <parent link="${name}arm_1_link"/>
+      <child link="${name}arm_2_link"/>
+    </joint>
+    <transmission name="${name}arm_1_trans" type="pr2_mechanism_model/SimpleTransmission">
+      <actuator name="${name}arm_1_motor"/>
+      <joint name="${name}arm_1_joint"/>
+      <mechanicalReduction>1.0</mechanicalReduction>
+    </transmission>
+    <link name="${name}arm_2_link">
       <inertial>
         <mass value="${arm_elem_link_mass}"/>
@@ -117,13 +122,8 @@
       </collision>
     </link>
-    <gazebo reference="${name}_arm_2_link">
-      <material value="kuka-lwr.material"/>
-    </gazebo>
-    <transmission name="${name}_arm_1_trans" type="pr2_mechanism_model/SimpleTransmission">
-      <actuator name="${name}_arm_1_motor"/>
-      <joint name="${name}_arm_1_joint"/>
-      <mechanicalReduction>1.0</mechanicalReduction>
-    </transmission>
-    <joint name="${name}_arm_2_joint" type="revolute">
+    <gazebo reference="${name}arm_2_link">
+      <material value="kuka-lwr.material"/>
+    </gazebo>
+    <joint name="${name}arm_2_joint" type="revolute">
       <origin xyz="0 0 0.20" rpy="0 0 0"/>
       <axis xyz="0 0 1"/>
@@ -135,8 +135,13 @@
                          k_velocity="${safety_controller_k_vel}"/>
       <dynamics damping="${joint_damping}"/>
-      <parent link="${name}_arm_2_link"/>
-      <child link="${name}_arm_3_link"/>
-    </joint>
-    <link name="${name}_arm_3_link">
+      <parent link="${name}arm_2_link"/>
+      <child link="${name}arm_3_link"/>
+    </joint>
+    <transmission name="${name}arm_2_trans" type="pr2_mechanism_model/SimpleTransmission">
+      <actuator name="${name}arm_2_motor"/>
+      <joint name="${name}arm_2_joint"/>
+      <mechanicalReduction>1.0</mechanicalReduction>
+    </transmission>
+    <link name="${name}arm_3_link">
       <inertial>
         <mass value="${arm_elem_link_mass}"/>
@@ -160,13 +165,8 @@
       </collision>
     </link>
-    <gazebo reference="${name}_arm_3_link">
-      <material value="kuka-lwr.material"/>
-    </gazebo>
-    <transmission name="${name}_arm_2_trans" type="pr2_mechanism_model/SimpleTransmission">
-      <actuator name="${name}_arm_2_motor"/>
-      <joint name="${name}_arm_2_joint"/>
-      <mechanicalReduction>1.0</mechanicalReduction>
-    </transmission>
-    <joint name="${name}_arm_3_joint" type="revolute">
+    <gazebo reference="${name}arm_3_link">
+      <material value="kuka-lwr.material"/>
+    </gazebo>
+    <joint name="${name}arm_3_joint" type="revolute">
       <origin xyz="0 0 0.20" rpy="0 0 0"/>
       <axis xyz="0 1 0"/>
@@ -178,8 +178,13 @@
                          k_velocity="${safety_controller_k_vel}"/>
       <dynamics damping="${joint_damping}"/>
-      <parent link="${name}_arm_3_link"/>
-      <child link="${name}_arm_4_link"/>
-    </joint>
-    <link name="${name}_arm_4_link">
+      <parent link="${name}arm_3_link"/>
+      <child link="${name}arm_4_link"/>
+    </joint>
+    <transmission name="${name}arm_3_trans" type="pr2_mechanism_model/SimpleTransmission">
+      <actuator name="${name}arm_3_motor"/>
+      <joint name="${name}arm_3_joint"/>
+      <mechanicalReduction>1.0</mechanicalReduction>
+    </transmission>
+    <link name="${name}arm_4_link">
       <inertial>
         <mass value="${arm_elem_link_mass}"/>
@@ -203,13 +208,8 @@
       </collision>
     </link>
-    <gazebo reference="${name}_arm_4_link">
-      <material value="kuka-lwr.material"/>
-    </gazebo>
-    <transmission name="${name}_arm_3_trans" type="pr2_mechanism_model/SimpleTransmission">
-      <actuator name="${name}_arm_3_motor"/>
-      <joint name="${name}_arm_3_joint"/>
-      <mechanicalReduction>1.0</mechanicalReduction>
-    </transmission>
-    <joint name="${name}_arm_4_joint" type="revolute">
+    <gazebo reference="${name}arm_4_link">
+      <material value="kuka-lwr.material"/>
+    </gazebo>
+    <joint name="${name}arm_4_joint" type="revolute">
       <origin xyz="0 0 0.20" rpy="0 0 0"/>
       <axis xyz="0 0 1"/>
@@ -221,8 +221,13 @@
                          k_velocity="${safety_controller_k_vel}"/>
       <dynamics damping="${joint_damping}"/>
-      <parent link="${name}_arm_4_link"/>
-      <child link="${name}_arm_5_link"/>
-    </joint>
-    <link name="${name}_arm_5_link">
+      <parent link="${name}arm_4_link"/>
+      <child link="${name}arm_5_link"/>
+    </joint>
+    <transmission name="${name}arm_4_trans" type="pr2_mechanism_model/SimpleTransmission">
+      <actuator name="${name}arm_4_motor"/>
+      <joint name="${name}arm_4_joint"/>
+      <mechanicalReduction>1.0</mechanicalReduction>
+    </transmission>
+    <link name="${name}arm_5_link">
       <inertial>
         <mass value="${arm_elem_link_mass}"/>
@@ -233,5 +238,5 @@
       <visual>
         <origin xyz="0 0 0" rpy="0 0 ${M_PI}"/>
-        <geometry name="${name}_arm_5_geom">
+        <geometry name="${name}arm_5_geom">
           <mesh scale="100 100 100"
 					 filename="package://agni_description/meshes/arm/arm_segment_last.dae"/>
@@ -246,13 +251,8 @@
       </collision>
     </link>
-    <gazebo reference="${name}_arm_5_link">
-      <material value="kuka-lwr.material"/>
-    </gazebo>
-    <transmission name="${name}_arm_4_trans" type="pr2_mechanism_model/SimpleTransmission">
-      <actuator name="${name}_arm_4_motor"/>
-      <joint name="${name}_arm_4_joint"/>
-      <mechanicalReduction>1.0</mechanicalReduction>
-    </transmission>
-    <joint name="${name}_arm_5_joint" type="revolute">
+    <gazebo reference="${name}arm_5_link">
+      <material value="kuka-lwr.material"/>
+    </gazebo>
+    <joint name="${name}arm_5_joint" type="revolute">
       <origin xyz="0 0 0.19" rpy="0 0 0"/>
       <axis xyz="0 -1 0"/>
@@ -264,8 +264,13 @@
                          k_velocity="${safety_controller_k_vel}"/>
       <dynamics damping="${joint_damping}"/>
-      <parent link="${name}_arm_5_link"/>
-      <child link="${name}_arm_6_link"/>
-    </joint>
-    <link name="${name}_arm_6_link">
+      <parent link="${name}arm_5_link"/>
+      <child link="${name}arm_6_link"/>
+    </joint>
+    <transmission name="${name}arm_5_trans" type="pr2_mechanism_model/SimpleTransmission">
+      <actuator name="${name}arm_5_motor"/>
+      <joint name="${name}arm_5_joint"/>
+      <mechanicalReduction>1.0</mechanicalReduction>
+    </transmission>
+    <link name="${name}arm_6_link">
       <inertial>
         <mass value="${arm_elem_ball_link_mass}"/>
@@ -289,13 +294,8 @@
       </collision>
     </link>
-    <gazebo reference="${name}_arm_6_link">
-      <material value="kuka-lwr.material"/>
-    </gazebo>
-    <transmission name="${name}_arm_5_trans" type="pr2_mechanism_model/SimpleTransmission">
-      <actuator name="${name}_arm_5_motor"/>
-      <joint name="${name}_arm_5_joint"/>
-      <mechanicalReduction>1.0</mechanicalReduction>
-    </transmission>
-    <joint name="${name}_arm_6_joint" type="revolute">
+    <gazebo reference="${name}arm_6_link">
+      <material value="kuka-lwr.material"/>
+    </gazebo>
+    <joint name="${name}arm_6_joint" type="revolute">
       <origin xyz="0 0 0.078" rpy="0 0 0"/>
       <axis xyz="0 0 1"/>
@@ -307,8 +307,13 @@
                          k_velocity="${safety_controller_k_vel}"/>
       <dynamics damping="${joint_damping}"/>
-      <parent link="${name}_arm_6_link"/>
-      <child link="${name}_arm_7_link"/>
-    </joint>
-    <link name="${name}_arm_7_link">
+      <parent link="${name}arm_6_link"/>
+      <child link="${name}arm_7_link"/>
+    </joint>
+    <transmission name="${name}arm_6_trans" type="pr2_mechanism_model/SimpleTransmission">
+      <actuator name="${name}arm_6_motor"/>
+      <joint name="${name}arm_6_joint"/>
+      <mechanicalReduction>1.0</mechanicalReduction>
+    </transmission>
+    <link name="${name}arm_7_link">
       <inertial>
         <mass value="${arm_elem_end_link_mass}"/>
@@ -332,21 +337,16 @@
       </collision>
     </link>
-    <gazebo reference="${name}_arm_7_link">
-      <material value="kuka-lwr.material"/>
-    </gazebo>
-    <transmission name="${name}_arm_6_trans" type="pr2_mechanism_model/SimpleTransmission">
-      <actuator name="${name}_arm_6_motor"/>
-      <joint name="${name}_arm_6_joint"/>
-      <mechanicalReduction>1.0</mechanicalReduction>
-    </transmission>
-    <joint name="${name}_arm_hand_fixed_joint" type="fixed">
+    <gazebo reference="${name}arm_7_link">
+      <material value="kuka-lwr.material"/>
+    </gazebo>
+    <joint name="${name}arm_hand_fixed_joint" type="fixed">
 <!--
       <origin xyz="${-right * 0.075} -0.075 -0.094"
               rpy="${0.5*right*M_PI} 0 ${(1.5 + 0.25*right)*M_PI}"/>
 -->
-      <parent link="${name}_arm_7_link"/>
-      <child link="${name}_arm_hand_link"/>
-    </joint>
-    <link name="${name}_arm_hand_link" />
+      <parent link="${name}arm_7_link"/>
+      <child link="${name}arm_hand_mount"/>
+    </joint>
+    <link name="${name}arm_hand_mount" />
   </macro>
 </robot>

File: urdf/test.urdf.xacro (robot description, xacro)
@@ -3,5 +3,6 @@
   <test value="${foo}"/>
   <xacro:property name="foo" value="0"/>
-  <xacro:if value="${-3*foo}"><no/></xacro:if>
+  <xacro:property name="bar" value="${1*foo}"/>
+  <xacro:if value="${-3*bar}"><no/></xacro:if>
   <xacro:if value="0"><no/></xacro:if>
   <xacro:if value="1"><yes/></xacro:if>
