Commit message: shortened PA10 frame, added mounting bar

File: robots/frame-pa10.urdf.xacro (robot description, xacro)
@@ -3,5 +3,26 @@
 		 xmlns:xacro="http://www.ros.org/wiki/xacro">
   <xacro:include filename="$(find agni_description)/urdf/frame.urdf.xacro"/>
-  <xacro:frame prefix="pa10" thickness="0.09" width="1.92" depth="1.82"
-					height="1.26" tableHeight="1.00"/>
+  <xacro:property name="thickness" value="0.09"/>
+  <xacro:property name="width" value="1.92"/>
+  <xacro:property name="depth" value="1.42"/>
+  <xacro:property name="height" value="2"/>
+  <xacro:property name="tableHeight" value="0.87"/>
+  <xacro:frame prefix="pa10" thickness="${thickness}"
+					width="${width}" depth="${depth}" height="${height}"
+					tableHeight="${tableHeight}"/>
+  <joint name="mounting" type="fixed">
+	 <parent link="pa10_frame"/>
+	 <child link="pa10_mounting"/>
+	 <origin xyz="0 0.85 1.12" rpy="0 0 0"/>
+  </joint>
+  <link name="pa10_mounting">
+	 <!-- front bar -->
+	 <xacro:bar thickness="${thickness}" len="${width}">
+		<origin xyz="0 ${-0.26-thickness/2} ${-thickness/2}" rpy="0 ${-M_PI/2} 0"/>
+	 </xacro:bar>
+	 <!-- rear bar -->
+	 <xacro:bar thickness="${thickness}" len="${width}">
+		<origin xyz="0 ${0.26+thickness/2} ${-thickness/2}" rpy="0 ${-M_PI/2} 0"/>
+	 </xacro:bar>
+  </link>
 </robot>
