Commit message: Added new launch files and urdf for kuka arm using controllers based on friComm Created specific launch files for gazebo to handle dual robots simulations

File: robots/kuka_hand_right_gazebo.urdf.xacro (robot description, xacro)
@@ -2,17 +2,32 @@
 <robot name="kuka_right"
 		 xmlns:xacro="http://www.ros.org/wiki/xacro">
+  <xacro:include filename="$(find agni_description)/calibration/default_cal.xml"/>
   <xacro:include filename="$(find agni_description)/kuka/lwr.urdf.xacro"/>
+  <xacro:include filename="$(find sr_description)/hand/xacro/full_hand_motor.urdf.xacro" />
+  <include filename="$(find sr_description)/other/xacro/gazebo/gazebo.urdf.xacro" />
   <!-- KUKA arms -->
   <xacro:kuka_lwr_arm name="right_" reflect="+1" tool_name=""/>
-  <link name="kuka_frame"/>
-  <joint name="right_frame_placement" type="fixed">
+  <link name="world" />
+  <link name="kuka_frame" />
+  <joint name="frame_placement" type="fixed">
+    <parent link="world"/>
+    <child link="kuka_frame"/>
+  </joint>
+  <joint name="right_arm_mount" type="fixed">
     <parent link="kuka_frame"/>
     <child link="right_arm_base_link"/>
+    <origin xyz="0.08 0.8 0.3" rpy="0 -1.047 0"/>
+  </joint>
+  <!-- Shadow Hands -->
+  <joint name="right_arm_hand_mount" type="fixed">
+    <parent link="right_arm_hand_mount"/>
+    <child link="forearm"/>
+    <origin xyz="0 0 0" rpy="0 0 0" />
   </joint>
   <gazebo>
-    <plugin name="right_lwr_controller" filename="liblwr_controller.so">
+    <plugin name="lwr_controller" filename="liblwr_controller.so">
       <alwaysOn>true</alwaysOn>
       <robotPrefix>right</robotPrefix>
-      <remotePort>49948</remotePort>
+      <remotePort>49938</remotePort>
       <baseLink>right_arm_base_link</baseLink>
       <toolLink>right_arm_hand_mount</toolLink>
@@ -26,3 +41,4 @@
     </plugin>
   </gazebo>
+  <xacro:shadowhand_motor/>
 </robot>

File: robots/kuka_left.urdf.xacro (robot description, xacro)
@@ -1,15 +1,8 @@
 <?xml version="1.0"?>
-<robot name="kukas"
+<robot name="kuka_left"
 		 xmlns:xacro="http://www.ros.org/wiki/xacro">
   <xacro:include filename="$(find agni_description)/calibration/default_cal.xml"/>
   <xacro:include filename="$(find agni_description)/kuka/lwr.urdf.xacro"/>
-  <xacro:include filename="$(find sr_description)/hand/xacro/full_hand_motor.urdf.xacro" />
-  <!-- KUKA arms -->
-  <xacro:kuka_lwr_arm name="left_" right="-1" tool_name=""/>
-  <joint name="left_arm_hand_mount" type="fixed">
-    <parent link="left_arm_hand_mount"/>
-    <child link="forearm"/>
-    <origin xyz="0 0 0" rpy="0 0 0" />
-  </joint>
-  <xacro:shadowhand_left_motor/>
+  <!-- KUKA arm -->
+  <xacro:kuka_lwr_arm name="left_" reflect="-1" tool_name=""/>
 </robot>

File: robots/kuka_right.urdf.xacro (robot description, xacro)
@@ -1,17 +1,7 @@
 <?xml version="1.0"?>
-<robot name="kukas"
+<robot name="kuka_right"
 		 xmlns:xacro="http://www.ros.org/wiki/xacro">
-  <xacro:include filename="$(find agni_description)/calibration/default_cal.xml"/>
   <xacro:include filename="$(find agni_description)/kuka/lwr.urdf.xacro"/>
-  <xacro:include filename="$(find sr_description)/hand/xacro/full_hand_motor.urdf.xacro" />
-  <include filename="$(find sr_description)/other/xacro/gazebo/gazebo.urdf.xacro" />
   <!-- KUKA arms -->
-  <xacro:kuka_lwr_arm name="right_" right="+1" tool_name=""/>
-  <!-- Shadow Hands -->
-  <joint name="right_arm_hand_mount" type="fixed">
-    <parent link="right_arm_hand_mount"/>
-    <child link="forearm"/>
-    <origin xyz="0 0 0" rpy="0 0 0" />
-  </joint>
-  <xacro:shadowhand_motor/>
+  <xacro:kuka_lwr_arm name="right_" reflect="+1" tool_name=""/>
 </robot>
