Commit message: PA10-a model

File: kuka/lwr.urdf.xacro (robot description, xacro)
@@ -26,5 +26,5 @@
         <geometry>
           <mesh scale="100 100 100"
-					 filename="package://agni_description/meshes/arm/arm_base.dae"/>
+					 filename="package://agni_description/kuka/meshes/arm_base.dae"/>
         </geometry>
         <material name="Orange"/>
@@ -33,5 +33,5 @@
         <origin xyz="0 0 0" rpy="0 0 0"/>
         <geometry>
-          <mesh filename="package://agni_description/meshes/arm/convex/arm_base_convex.stl"/>
+          <mesh filename="package://agni_description/kuka/meshes/convex/arm_base_convex.stl"/>
         </geometry>
       </collision>
@@ -68,12 +68,12 @@
         <origin xyz="0 0 0" rpy="0 0 ${M_PI}"/>
         <geometry>
-          <mesh scale="100 100 100"  filename="package://agni_description/meshes/arm/arm_segment_a.dae"/>
-        </geometry>
-        <material name="Orange"/>
-      </visual>
-      <collision>
-        <origin xyz="0 0 0" rpy="0 0 ${M_PI}"/>
-        <geometry>
-          <mesh filename="package://agni_description/meshes/arm/convex/arm_segment_a_convex.stl"/>
+          <mesh scale="100 100 100"  filename="package://agni_description/kuka/meshes/arm_segment_a.dae"/>
+        </geometry>
+        <material name="Orange"/>
+      </visual>
+      <collision>
+        <origin xyz="0 0 0" rpy="0 0 ${M_PI}"/>
+        <geometry>
+          <mesh filename="package://agni_description/kuka/meshes/convex/arm_segment_a_convex.stl"/>
         </geometry>
       </collision>
@@ -111,5 +111,5 @@
         <geometry>
           <mesh scale="100 100 100"
-					 filename="package://agni_description/meshes/arm/arm_segment_b.dae"/>
+					 filename="package://agni_description/kuka/meshes/arm_segment_b.dae"/>
         </geometry>
         <material name="Orange"/>
@@ -118,5 +118,5 @@
         <origin xyz="0 0 0.2" rpy="${M_PI} 0 ${M_PI}"/>
         <geometry>
-          <mesh filename="package://agni_description/meshes/arm/convex/arm_segment_b_convex.stl"/>
+          <mesh filename="package://agni_description/kuka/meshes/convex/arm_segment_b_convex.stl"/>
         </geometry>
       </collision>
@@ -154,5 +154,5 @@
         <geometry>
           <mesh scale="100 100 100"
-					 filename="package://agni_description/meshes/arm/arm_segment_a.dae"/>
+					 filename="package://agni_description/kuka/meshes/arm_segment_a.dae"/>
         </geometry>
         <material name="Orange"/>
@@ -161,5 +161,5 @@
         <origin xyz="0 0 0" rpy="0 0 0"/>
         <geometry>
-          <mesh filename="package://agni_description/meshes/arm/convex/arm_segment_a_convex.stl"/>
+          <mesh filename="package://agni_description/kuka/meshes/convex/arm_segment_a_convex.stl"/>
         </geometry>
       </collision>
@@ -197,5 +197,5 @@
         <geometry>
           <mesh scale="100 100 100"
-					 filename="package://agni_description/meshes/arm/arm_segment_b.dae"/>
+					 filename="package://agni_description/kuka/meshes/arm_segment_b.dae"/>
         </geometry>
         <material name="Orange"/>
@@ -204,5 +204,5 @@
         <origin xyz="0 0 0.2" rpy="0 ${M_PI} ${M_PI}"/>
         <geometry>
-          <mesh filename="package://agni_description/meshes/arm/convex/arm_segment_b_convex.stl"/>
+          <mesh filename="package://agni_description/kuka/meshes/convex/arm_segment_b_convex.stl"/>
         </geometry>
       </collision>
@@ -240,12 +240,12 @@
         <geometry name="${name}arm_5_geom">
           <mesh scale="100 100 100"
-					 filename="package://agni_description/meshes/arm/arm_segment_last.dae"/>
-        </geometry>
-        <material name="Orange"/>
-      </visual>
-      <collision>
-        <origin xyz="0 0 0" rpy="0 0 ${M_PI}"/>
-        <geometry>
-          <mesh filename="package://agni_description/meshes/arm/convex/arm_segment_last_convex.stl"/>
+					 filename="package://agni_description/kuka/meshes/arm_segment_last.dae"/>
+        </geometry>
+        <material name="Orange"/>
+      </visual>
+      <collision>
+        <origin xyz="0 0 0" rpy="0 0 ${M_PI}"/>
+        <geometry>
+          <mesh filename="package://agni_description/kuka/meshes/convex/arm_segment_last_convex.stl"/>
         </geometry>
       </collision>
@@ -283,5 +283,5 @@
         <geometry>
           <mesh scale="100 100 100"
-					 filename="package://agni_description/meshes/arm/arm_wrist.dae"/>
+					 filename="package://agni_description/kuka/meshes/arm_wrist.dae"/>
         </geometry>
         <material name="Grey"/>
@@ -290,5 +290,5 @@
         <origin xyz="0 0 0" rpy="0 0 ${M_PI}"/>
         <geometry>
-          <mesh filename="package://agni_description/meshes/arm/convex/arm_wrist_convex.stl"/>
+          <mesh filename="package://agni_description/kuka/meshes/convex/arm_wrist_convex.stl"/>
         </geometry>
       </collision>
@@ -326,5 +326,5 @@
         <geometry>
           <mesh scale="100 100 100"
-					 filename="package://agni_description/meshes/arm/arm_flanche${tool_name}.dae"/>
+					 filename="package://agni_description/kuka/meshes/arm_flanche${tool_name}.dae"/>
         </geometry>
         <material name="Grey"/>
@@ -333,5 +333,5 @@
         <origin xyz="0 0 0" rpy="0 0 ${right * -1/4 * M_PI  +  M_PI}"/>
         <geometry>
-          <mesh filename="package://agni_description/meshes/arm/convex/arm_flanche${tool_name}_convex.stl"/>
+          <mesh filename="package://agni_description/kuka/meshes/convex/arm_flanche${tool_name}_convex.stl"/>
         </geometry>
       </collision>

File: shadow/forearm.urdf.xacro (robot description, xacro)
@@ -1,5 +1,5 @@
 <robot xmlns:xacro="http://ros.org/wiki/xacro">
-  <xacro:macro name="shadow_hand_forearm">
-    <link name="${name}hand_forearm">
+  <xacro:macro name="forearm">
+    <link name="${prefix}forearm">
       <inertial>
 		  <origin xyz="0 0 0.09" rpy="0 0 0"/>
@@ -9,6 +9,7 @@
       <visual>
 		  <origin xyz="0 0 0" rpy="0 0 0" />
-		  <geometry name="shadow_forearm_geom">
-			 <mesh filename="package://sr_description/hand/model/forearm.dae" scale="0.001 0.001 0.001"/>
+		  <geometry name="forearm">
+			 <mesh filename="package://agni_description/shadow/meshes/forearm.dae"
+					 scale="0.001 0.001 0.001"/>
 		  </geometry>
 		  <material name="Grey" />
@@ -16,10 +17,10 @@
       <collision>
 		  <origin xyz="0 0 0.09" rpy="0 0 0" />
-		  <geometry name="shadow_forearm_collision">
+		  <geometry name="forearm">
 			 <cylinder radius="0.06" length="0.180"/>
 		  </geometry>
       </collision>
     </link>
-    <gazebo reference="${name}hand_forearm">
+    <gazebo reference="${prefix}forearm">
       <material>Gazebo/Grey</material>
       <selfCollide>false</selfCollide>

Commit message: Changes by QLI to be tested

File: kuka/lwr.urdf.xacro (robot description, xacro)
@@ -13,6 +13,6 @@
   <property name="joint_damping" value="0.1" />
   <property name="arm_velocity_scale_factor" value="1"/>
-  <!-- right is either 1 (for right arm) or -1 (for left arm) -->
-  <macro name="kuka_lwr_arm" params="name right tool_name">
+  <!-- reflect is either 1 (for right arm) or -1 (for left arm) -->
+  <macro name="kuka_lwr_arm" params="name reflect tool_name">
     <link name="${name}arm_base_link">
       <inertial>
@@ -323,5 +323,5 @@
       </inertial>
       <visual>
-        <origin xyz="0 0 0" rpy="0 0 ${right * -1/4 * M_PI  +  M_PI}"/>
+        <origin xyz="0 0 0" rpy="0 0 ${reflect * -1/4 * M_PI  +  M_PI}"/>
         <geometry>
           <mesh scale="100 100 100"
@@ -331,5 +331,5 @@
       </visual>
       <collision>
-        <origin xyz="0 0 0" rpy="0 0 ${right * -1/4 * M_PI  +  M_PI}"/>
+        <origin xyz="0 0 0" rpy="0 0 ${reflect * -1/4 * M_PI  +  M_PI}"/>
         <geometry>
           <mesh filename="package://agni_description/kuka/meshes/convex/arm_flanche${tool_name}_convex.stl"/>
@@ -342,6 +342,6 @@
     <joint name="${name}arm_hand_fixed_joint" type="fixed">
 <!--
-      <origin xyz="${-right * 0.075} -0.075 -0.094"
-              rpy="${0.5*right*M_PI} 0 ${(1.5 + 0.25*right)*M_PI}"/>
+      <origin xyz="${-reflect * 0.075} -0.075 -0.094"
+              rpy="${0.5*reflect*M_PI} 0 ${(1.5 + 0.25*reflect)*M_PI}"/>
 -->
       <parent link="${name}arm_7_link"/>

File: robots/kuka_right.urdf.xacro (robot description, xacro)
@@ -5,4 +5,5 @@
   <xacro:include filename="$(find agni_description)/kuka/lwr.urdf.xacro"/>
   <xacro:include filename="$(find sr_description)/hand/xacro/full_hand_motor.urdf.xacro" />
+  <include filename="$(find sr_description)/other/xacro/gazebo/gazebo.urdf.xacro" />
   <!-- KUKA arms -->
   <xacro:kuka_lwr_arm name="right_" right="+1" tool_name=""/>

File: robots/kukas.urdf.xacro (robot description, xacro)
@@ -5,34 +5,36 @@
   <xacro:include filename="$(find agni_description)/urdf/frame-half.urdf.xacro"/>
   <xacro:include filename="$(find agni_description)/kuka/lwr.urdf.xacro"/>
-  <xacro:include filename="$(find sr_description)/hand/xacro/full_hand_motor.urdf.xacro" />
+  <xacro:include filename="$(find sr_description)/hand/xacro/full_hand.urdf.xacro" />
   <xacro:frame-half prefix="kuka" thickness="0.09" width="1.92" depth="1.82"
 						  height="1.26" tableHeight="1.00"/>
   <!-- KUKA arms -->
-  <xacro:kuka_lwr_arm name="right" right="+1" tool_name=""/>
+  <xacro:kuka_lwr_arm name="right_" reflect="+1" tool_name=""/>
   <joint name="kuka_right_arm_base_joint" type="fixed">
 	 <origin xyz="${cal_right_arm_x} ${cal_right_arm_y} ${cal_right_arm_z}"
 				rpy="${cal_right_arm_roll} ${cal_right_arm_pitch} ${cal_right_arm_yaw}"/>
 	 <parent link="kuka_frame"/>
-	 <child link="calib_right_arm_base_link"/>
+	 <child link="right_arm_base_link"/>
+	<!-- <child link="calib_right_arm_base_link"/> -->
   </joint>
-  <xacro:kuka_lwr_arm name="left" right="-1" tool_name=""/>
+  <xacro:kuka_lwr_arm name="left_" reflect="-1" tool_name=""/>
   <joint name="kuka_left_arm_base_joint" type="fixed">
 	 <origin xyz="${cal_left_arm_x} ${cal_left_arm_y} ${cal_left_arm_z}"
 				rpy="${cal_left_arm_roll} ${cal_left_arm_pitch} ${cal_left_arm_yaw}"/>
 	 <parent link="kuka_frame"/>
-	 <child link="calib_left_arm_base_link"/>
+	 <child link="left_arm_base_link"/>
+	<!-- <child link="calib_left_arm_base_link"/> -->
   </joint>
   <!-- Shadow Hands -->
+  <xacro:shadowhand muscletrans="false" muscle="false" bio="false" ubi="true" eli="false" reflect="-1.0" prefix="l_" />
   <joint name="left_arm_hand_mount" type="fixed">
     <parent link="left_arm_hand_mount"/>
-    <child link="forearm"/>
-    <origin xyz="0 0 0" rpy="0 0 ${2.35619449}" />
+    <child link="l_forearm"/>
+    <origin xyz="0 0 0" rpy="0 0 0" />
   </joint>
-  <xacro:shadowhand_left_motor/>
+  <xacro:shadowhand muscletrans="false" muscle="false" bio="false" ubi="true" eli="false" reflect="1.0" prefix="r_"  />
   <joint name="right_arm_hand_mount" type="fixed">
     <parent link="right_arm_hand_mount"/>
-    <child link="forearm"/>
+    <child link="r_forearm"/>
     <origin xyz="0 0 0" rpy="0 0 0" />
   </joint>
-  <xacro:shadowhand_motor/>
 </robot>

File: urdf/frame-half.urdf.xacro (robot description, xacro)
@@ -1,4 +1,7 @@
 <?xml version="1.0"?>
-<root xmlns:xacro="http://www.ros.org/wiki/xacro">
+<root xmlns:xacro="http://www.ros.org/wiki/xacro"
+      xmlns:sensor="http://playerstage.sourceforge.net/gazebo/xmlschema/#sensor"
+      xmlns:controller="http://playerstage.sourceforge.net/gazebo/xmlschema/#controller"
+      xmlns:interface="http://playerstage.sourceforge.net/gazebo/xmlschema/#interface">
 <xacro:include filename="$(find agni_description)/urdf/util.urdf.xacro"/>
 <xacro:include filename="$(find agni_description)/urdf/materials.urdf.xacro"/>
@@ -51,4 +54,7 @@
 	 </xacro:bar>
   </link>
+  <gazebo reference="${prefix}_frame">
+      <material value="kuka-lwr.material"/>
+  </gazebo>
 </xacro:macro>
 </root>
