Commit message: Improved hand and arm launch files with cleaner upload/bringup/controllers launchers Added sr_gazebo_controller_manager launcher in a namespace Fixed rk/lk deploy Now Right and Left arm+hand working (no joint_states merging yet)

File: agni_description/robots/lh_ubi_motor_hand.urdf.xacro (robot description, xacro)
@@ -4,5 +4,6 @@
 	<xacro:include filename="$(find sr_description)/materials.urdf.xacro" />
   <xacro:include filename="$(find sr_description)/hand/xacro/full_hand.urdf.xacro" />
-  <xacro:include filename="$(find sr_description)/other/xacro/gazebo/gazebo.urdf.xacro" />
+  <xacro:include filename="$(find agni_description)/urdf/sr_gazebo.urdf.xacro" />
+  <xacro:shadow_gazebo_controller_manager namespace="lh" />
   <xacro:shadowhand muscletrans="false" muscle="false" bio="false" ubi="true" eli="false" reflect="-1.0" prefix=""  />
 </robot>

File: agni_description/robots/lh_ubi_motor_hand_prefix.urdf.xacro (robot description, xacro)
@@ -4,5 +4,6 @@
 	<xacro:include filename="$(find sr_description)/materials.urdf.xacro" />
   <xacro:include filename="$(find sr_description)/hand/xacro/full_hand.urdf.xacro" />
-  <xacro:include filename="$(find sr_description)/other/xacro/gazebo/gazebo.urdf.xacro" />
+  <xacro:include filename="$(find agni_description)/urdf/sr_gazebo.urdf.xacro" />
+  <xacro:shadow_gazebo_controller_manager namespace="rh" />
   <xacro:shadowhand muscletrans="false" muscle="false" bio="false" ubi="true" eli="false" reflect="-1.0" prefix="l_"  />
 </robot>

File: agni_description/robots/lk_kuka_gazebo.urdf.xacro (robot description, xacro)
@@ -3,27 +3,7 @@
 		 xmlns:xacro="http://www.ros.org/wiki/xacro">
   <xacro:include filename="$(find agni_description)/kuka/lwr.urdf.xacro"/>
-  <!-- KUKA arms -->
+  <xacro:include filename="$(find agni_description)/kuka/lwr_controllers.gazebo.xacro"/>
+  <!-- KUKA arm -->
   <xacro:kuka_lwr_arm name="left_" reflect="-1" tool_name=""/>
-  <link name="kuka_frame"/>
-  <joint name="left_frame_placement" type="fixed">
-    <parent link="kuka_frame"/>
-    <child link="left_arm_base_link"/>
-  </joint>
-  <gazebo>
-    <plugin name="left_lwr_arm_controller" filename="liblwr_controller.so">
-      <alwaysOn>true</alwaysOn>
-      <robotPrefix>left</robotPrefix>
-      <robotNamespace>lk</robotNamespace>
-      <remotePort>49938</remotePort>
-      <baseLink>left_arm_base_link</baseLink>
-      <toolLink>left_arm_hand_mount</toolLink>
-      <left_arm_0_joint>0.0</left_arm_0_joint>
-      <left_arm_1_joint>0</left_arm_1_joint>
-      <left_arm_2_joint>0.0</left_arm_2_joint>
-      <left_arm_3_joint>0</left_arm_3_joint>
-      <left_arm_4_joint>0</left_arm_4_joint>
-      <left_arm_5_joint>0</left_arm_5_joint>
-      <left_arm_6_joint>0</left_arm_6_joint>
-    </plugin>
-  </gazebo>
+  <xacro:left_lwr_arm_gazebo_controller namespace="lk" port="49938"/>
 </robot>

File: agni_description/robots/rh_ubi_motor_hand.urdf.xacro (robot description, xacro)
@@ -4,5 +4,6 @@
 	<xacro:include filename="$(find sr_description)/materials.urdf.xacro" />
   <xacro:include filename="$(find sr_description)/hand/xacro/full_hand.urdf.xacro" />
-  <xacro:include filename="$(find sr_description)/other/xacro/gazebo/gazebo.urdf.xacro" />
+  <xacro:include filename="$(find agni_description)/urdf/sr_gazebo.urdf.xacro" />
+  <xacro:shadow_gazebo_controller_manager namespace="rh" />
   <xacro:shadowhand muscletrans="false" muscle="false" bio="false" ubi="true" eli="false" reflect="1.0" prefix=""  />
 </robot>

File: agni_description/robots/rh_ubi_motor_hand_prefix.urdf.xacro (robot description, xacro)
@@ -4,5 +4,6 @@
 	<xacro:include filename="$(find sr_description)/materials.urdf.xacro" />
   <xacro:include filename="$(find sr_description)/hand/xacro/full_hand.urdf.xacro" />
-  <xacro:include filename="$(find sr_description)/other/xacro/gazebo/gazebo.urdf.xacro" />
+  <xacro:include filename="$(find agni_description)/urdf/sr_gazebo.urdf.xacro" />
+  <xacro:shadow_gazebo_controller_manager namespace="rh" />
   <xacro:shadowhand muscletrans="false" muscle="false" bio="false" ubi="true" eli="false" reflect="1.0" prefix="r_"  />
 </robot>

File: agni_description/robots/rk_kuka_gazebo.urdf.xacro (robot description, xacro)
@@ -3,27 +3,7 @@
 		 xmlns:xacro="http://www.ros.org/wiki/xacro">
   <xacro:include filename="$(find agni_description)/kuka/lwr.urdf.xacro"/>
-  <!-- KUKA arms -->
+  <xacro:include filename="$(find agni_description)/kuka/lwr_controllers.gazebo.xacro"/>
+  <!-- KUKA arm -->
   <xacro:kuka_lwr_arm name="right_" reflect="1" tool_name=""/>
-  <link name="kuka_frame"/>
-  <joint name="right_frame_placement" type="fixed">
-    <parent link="kuka_frame"/>
-    <child link="right_arm_base_link"/>
-  </joint>
-  <gazebo>
-    <plugin name="right_lwr_arm_controller" filename="liblwr_controller.so">
-      <alwaysOn>true</alwaysOn>
-      <robotPrefix>right</robotPrefix>
-      <robotNamespace>rk</robotNamespace>
-      <remotePort>49940</remotePort>
-      <baseLink>right_arm_base_link</baseLink>
-      <toolLink>right_arm_hand_mount</toolLink>
-      <right_arm_0_joint>0.0</right_arm_0_joint>
-      <right_arm_1_joint>0</right_arm_1_joint>
-      <right_arm_2_joint>0.0</right_arm_2_joint>
-      <right_arm_3_joint>0</right_arm_3_joint>
-      <right_arm_4_joint>0</right_arm_4_joint>
-      <right_arm_5_joint>0</right_arm_5_joint>
-      <right_arm_6_joint>0</right_arm_6_joint>
-    </plugin>
-  </gazebo>
+  <xacro:right_lwr_arm_gazebo_controller namespace="rk" port="49940"/>
 </robot>

File: agni_description/urdf/gazebo.urdf.xacro (robot description, xacro)
@@ -6,4 +6,4 @@
       <updateRate>1000.0</updateRate>
     </plugin>
-      </gazebo>
+  </gazebo>
 </robot>
