Commit message: Changed calibration file for kuka arm base link to reflect current setup Added the shadow mounting bracket space betwween kuka and hand Fixed the kuka frame

File: agni_description/robots/kukas.urdf.xacro (robot description, xacro)
@@ -30,5 +30,5 @@
     <parent link="left_arm_hand_mount"/>
     <child link="l_forearm"/>
-    <origin xyz="0 0 0" rpy="0 0 0" />
+    <origin xyz="0 0 0.0151" rpy="0 0 0" />
   </joint>
   <xacro:shadowhand muscletrans="false" muscle="false" bio="false" ubi="true" eli="false" reflect="1.0" prefix="r_"  />
@@ -36,5 +36,5 @@
     <parent link="right_arm_hand_mount"/>
     <child link="r_forearm"/>
-    <origin xyz="0 0 0" rpy="0 0 0" />
+    <origin xyz="0 0 0.0151" rpy="0 0 0" />
   </joint>
 </robot>

File: agni_description/urdf/frame-half.urdf.xacro (robot description, xacro)
@@ -17,5 +17,5 @@
 	 <!-- horizontal front bar-->
 	 <xacro:bar thickness="${thickness}" len="${width}">
-		<origin xyz="0 ${-thickness/2} ${-thickness/2}" rpy="0 ${-M_PI/2} 0"/>
+		<origin xyz="0 ${thickness/2} ${-thickness/2}" rpy="0 ${-M_PI/2} 0"/>
 	 </xacro:bar>
 	 <!-- horizontal rear bar -->
@@ -29,9 +29,9 @@
 	 <!-- left front pole -->
 	 <xacro:bar thickness="${thickness}" len="${thickness+tableHeight}">
-		<origin xyz="${-(width+thickness)/2} ${-thickness/2} ${-(thickness+tableHeight)/2}"/>
+		<origin xyz="${-(width+thickness)/2} ${thickness/2} ${-(thickness+tableHeight)/2}"/>
 	 </xacro:bar>
 	 <!-- right front pole -->
 	 <xacro:bar thickness="${thickness}" len="${thickness+tableHeight}">
-		<origin xyz="${+(width+thickness)/2} ${-thickness/2} ${-(thickness+tableHeight)/2}"/>
+		<origin xyz="${+(width+thickness)/2} ${thickness/2} ${-(thickness+tableHeight)/2}"/>
 	 </xacro:bar>
 	 <!-- left rear pole -->
@@ -53,4 +53,19 @@
 				  rpy="${-M_PI/2} 0 0"/>
 	 </xacro:bar>
+	 <!-- left central pole -->
+	 <xacro:bar thickness="${thickness}" len="${thickness+tableHeight+(height)/2}">
+		<origin xyz="${-thickness} ${(depth)/2+2*thickness} ${-(2*tableHeight-height)/4-thickness/2}"/>
+	 </xacro:bar>
+	 <!-- right central pole -->
+	 <xacro:bar thickness="${thickness}" len="${thickness+tableHeight+(height)/2}">
+		<origin xyz="${thickness} ${(depth)/2+2*thickness} ${-(2*tableHeight-height)/4-thickness/2}"/>
+	 </xacro:bar>
+	<!-- table plane -->
+	 <visual>
+	  <origin xyz="0 ${depth/2} -0.01"
+				  rpy="0 0 0"/>
+		<geometry><box size="${width} ${depth} ${0.02}"/></geometry>
+		<material name="Silver"/>
+	 </visual>
   </link>
   <gazebo reference="${prefix}_frame">
