Commit message: cleanup, removing unused files and renaming kukas to kuka_shadow Added the shadow mounting bracket

File: agni_description/robots/both_kuka_shadow.urdf.xacro (robot description, xacro)
@@ -1,4 +1,4 @@
 <?xml version="1.0"?>
-<robot name="kukas"
+<robot name="kuka_shadow"
 		 xmlns:xacro="http://www.ros.org/wiki/xacro">
   <xacro:include filename="$(find agni_description)/calibration/default_cal.xml"/>

File: agni_description/robots/left_kuka_shadow_gazebo.urdf.xacro (robot description, xacro)
@@ -1,4 +1,4 @@
 <?xml version="1.0"?>
-<robot name="left_kukas"
+<robot name="left_kuka_shadow"
 		 xmlns:xacro="http://www.ros.org/wiki/xacro">
   <xacro:include filename="$(find agni_description)/kuka/lwr.urdf.xacro"/>

File: agni_description/robots/right_kuka_shadow_gazebo.urdf.xacro (robot description, xacro)
@@ -1,4 +1,4 @@
 <?xml version="1.0"?>
-<robot name="right_kukas"
+<robot name="right_kuka_shadow"
 		 xmlns:xacro="http://www.ros.org/wiki/xacro">
   <xacro:include filename="$(find agni_description)/kuka/lwr.urdf.xacro"/>
@@ -24,5 +24,5 @@
     <parent link="right_arm_hand_mount"/>
     <child link="r_forearm"/>
-    <origin xyz="0 0 0" rpy="0 0 0" />
+    <origin xyz="0 0 0.0151" rpy="0 0 0" />
   </joint>
 </robot>
