Commit message: Added use_prefix arguments to handle prefixing or not (reduces number of files) Changed file names to use shadow and kuka as later as possible to remain generic (and maybe switch arm to pa-10 later) Fixed a typo in a xacro file (rh instead of lh)

File: agni_description/robots/left_kuka_shadow_prefix_gazebo.urdf.xacro (robot description, xacro)
@@ -18,10 +18,10 @@
   <xacro:left_lwr_arm_gazebo_controller namespace="lk" port="49938"/>
   <!-- Shadow hand -->
-	<xacro:shadowhand muscletrans="false" muscle="false" bio="false" ubi="true" eli="false" reflect="-1.0" prefix="" />
+	<xacro:shadowhand muscletrans="false" muscle="false" bio="false" ubi="true" eli="false" reflect="-1.0" prefix="l_" />
 	<xacro:shadow_gazebo_controller_manager namespace="lh" />
 	<!-- Link arm and hand -->
   <joint name="left_arm_hand_mount" type="fixed">
     <parent link="left_arm_hand_mount"/>
-    <child link="forearm"/>
+    <child link="l_forearm"/>
     <origin xyz="0 0 0" rpy="0 0 0" />
   </joint>

File: agni_description/robots/lh_ubi_motor_hand_prefix.urdf.xacro (robot description, xacro)
@@ -5,5 +5,5 @@
   <xacro:include filename="$(find sr_description)/hand/xacro/full_hand.urdf.xacro" />
   <xacro:include filename="$(find agni_description)/urdf/sr_gazebo.urdf.xacro" />
-  <xacro:shadow_gazebo_controller_manager namespace="rh" />
+  <xacro:shadow_gazebo_controller_manager namespace="lh" />
   <xacro:shadowhand muscletrans="false" muscle="false" bio="false" ubi="true" eli="false" reflect="-1.0" prefix="l_"  />
 </robot>

File: agni_description/robots/right_kuka_shadow_prefix_gazebo.urdf.xacro (robot description, xacro)
@@ -18,10 +18,10 @@
   <xacro:right_lwr_arm_gazebo_controller namespace="rk" port="49940"/>
   <!-- Shadow Hands -->
-  <xacro:shadowhand muscletrans="false" muscle="false" bio="false" ubi="true" eli="false" reflect="1.0" prefix=""  />
+  <xacro:shadowhand muscletrans="false" muscle="false" bio="false" ubi="true" eli="false" reflect="1.0" prefix="r_"  />
   <xacro:shadow_gazebo_controller_manager namespace="rh" />
   <!-- Link arm and hand -->
   <joint name="right_arm_hand_mount" type="fixed">
     <parent link="right_arm_hand_mount"/>
-    <child link="forearm"/>
+    <child link="r_forearm"/>
     <origin xyz="0 0 0.0151" rpy="0 0 0" />
   </joint>
