Commit message: Added Flobi head and nested a little more arm_and_hand robot Added missing elements on the frame (triangle, collision elements)

File: agni_description/robots/both_kuka_shadow_flobi.urdf.xacro (robot description, xacro)
@@ -1,4 +1,4 @@
 <?xml version="1.0"?>
-<robot name="kuka_shadow"
+<robot name="kuka_shadow_flobi"
      xmlns:xacro="http://www.ros.org/wiki/xacro">
   <xacro:include filename="$(find agni_description)/robots/right_kuka_shadow.urdf.xacro" />
@@ -6,4 +6,5 @@
   <xacro:include filename="$(find agni_description)/calibration/default_cal.xml"/>
   <xacro:include filename="$(find agni_description)/urdf/frame-half.urdf.xacro"/>
+  <xacro:include filename="$(find agni_description)/flobi/flobiv3.urdf.xacro" />
   <xacro:frame-half prefix="kuka" thickness="0.09" width="1.92" depth="1.82"
               height="1.26" tableHeight="1.00"/>
@@ -17,3 +18,6 @@
         rpy="${cal_left_arm_roll} ${cal_left_arm_pitch} ${cal_left_arm_yaw}"/>
   </xacro:leftkukashadow>
+  <xacro:flobi prefix="" neutral="1" gender="0" parent="kuka_frame" >
+		<origin xyz="0 ${cal_right_arm_y} ${cal_right_arm_z+mount_triangle_length/2*sin60+0.01}" rpy="0 0 ${-M_PI/2}"/>
+  </xacro:flobi>
 </robot>

File: agni_description/robots/left_kuka_shadow_gazebo.urdf.xacro (robot description, xacro)
@@ -2,27 +2,11 @@
 <robot name="left_kuka_shadow"
 		 xmlns:xacro="http://www.ros.org/wiki/xacro">
-  <xacro:include filename="$(find agni_description)/kuka/lwr.urdf.xacro"/>
-  <xacro:include filename="$(find agni_description)/kuka/lwr_controllers.gazebo.xacro"/>
-  <xacro:include filename="$(find agni_description)/urdf/sr_gazebo.urdf.xacro" />
-  <xacro:include filename="$(find sr_description)/hand/xacro/full_hand.urdf.xacro" />
+  <xacro:include filename="$(find agni_description)/robots/left_kuka_shadow.urdf.xacro" />
   <xacro:include filename="$(find agni_description)/calibration/default_cal.xml"/>
-   <link name="world" />
-  <!-- KUKA arm -->
-  <xacro:kuka_lwr_arm name="left_" reflect="-1" tool_name=""/>
-   <joint name="left_frame_placement" type="fixed">
-	 <origin xyz="${cal_left_arm_x} ${cal_left_arm_y} ${cal_left_arm_z}"
+  <link name="world" />
+  <!-- KUKA Shadow arm and hand  -->
+  <xacro:leftkukashadow parent="world" prefix="false" controller="true">
+    <origin xyz="${cal_left_arm_x} ${cal_left_arm_y} ${cal_left_arm_z}"
 				rpy="${cal_left_arm_roll} ${cal_left_arm_pitch} ${cal_left_arm_yaw}"/>
-	 <parent link="world"/>
-	 <child link="left_arm_base_link"/>
-  </joint>
-  <xacro:left_lwr_arm_gazebo_controller namespace="lk" port="49938"/>
-  <!-- Shadow hand -->
-	<xacro:shadowhand muscletrans="false" muscle="false" bio="false" ubi="true" eli="false" reflect="-1.0" prefix="" />
-	<xacro:shadow_gazebo_controller_manager namespace="lh" />
-	<!-- Link arm and hand -->
-  <joint name="left_arm_hand_mount" type="fixed">
-    <parent link="left_arm_hand_mount"/>
-    <child link="forearm"/>
-    <origin xyz="0 0 0" rpy="0 0 0" />
-  </joint>
+  </xacro:leftkukashadow>
 </robot>

File: agni_description/robots/left_kuka_shadow_prefix_gazebo.urdf.xacro (robot description, xacro)
@@ -1,28 +1,11 @@
 <?xml version="1.0"?>
 <robot name="left_kuka_shadow"
-		 xmlns:xacro="http://www.ros.org/wiki/xacro">
-  <xacro:include filename="$(find agni_description)/kuka/lwr.urdf.xacro"/>
-  <xacro:include filename="$(find agni_description)/kuka/lwr_controllers.gazebo.xacro"/>
-  <xacro:include filename="$(find agni_description)/urdf/sr_gazebo.urdf.xacro" />
-  <xacro:include filename="$(find sr_description)/hand/xacro/full_hand.urdf.xacro" />
+  <xacro:include filename="$(find agni_description)/robots/left_kuka_shadow.urdf.xacro" />
   <xacro:include filename="$(find agni_description)/calibration/default_cal.xml"/>
-   <link name="world" />
-  <!-- KUKA arm -->
-  <xacro:kuka_lwr_arm name="left_" reflect="-1" tool_name=""/>
-   <joint name="left_frame_placement" type="fixed">
-	 <origin xyz="${cal_left_arm_x} ${cal_left_arm_y} ${cal_left_arm_z}"
+  <link name="world" />
+  <!-- KUKA Shadow arm and hand  -->
+  <xacro:leftkukashadow parent="world" prefix="true" controller="true">
+    <origin xyz="${cal_left_arm_x} ${cal_left_arm_y} ${cal_left_arm_z}"
 				rpy="${cal_left_arm_roll} ${cal_left_arm_pitch} ${cal_left_arm_yaw}"/>
-	 <parent link="world"/>
-	 <child link="left_arm_base_link"/>
-  </joint>
-  <xacro:left_lwr_arm_gazebo_controller namespace="lk" port="49938"/>
-  <!-- Shadow hand -->
-	<xacro:shadowhand muscletrans="false" muscle="false" bio="false" ubi="true" eli="false" reflect="-1.0" prefix="l_" />
-	<xacro:shadow_gazebo_controller_manager namespace="lh" />
-	<!-- Link arm and hand -->
-  <joint name="left_arm_hand_mount" type="fixed">
-    <parent link="left_arm_hand_mount"/>
-    <child link="l_forearm"/>
-    <origin xyz="0 0 0" rpy="0 0 0" />
-  </joint>
+  </xacro:leftkukashadow>
 </robot>

File: agni_description/robots/right_kuka_shadow_gazebo.urdf.xacro (robot description, xacro)
@@ -1,28 +1,12 @@
 <?xml version="1.0"?>
 <robot name="right_kuka_shadow"
-		 xmlns:xacro="http://www.ros.org/wiki/xacro">
-  <xacro:include filename="$(find agni_description)/kuka/lwr.urdf.xacro"/>
-  <xacro:include filename="$(find agni_description)/kuka/lwr_controllers.gazebo.xacro"/>
-  <xacro:include filename="$(find agni_description)/urdf/sr_gazebo.urdf.xacro" />
-  <xacro:include filename="$(find sr_description)/hand/xacro/full_hand.urdf.xacro" />
-   <xacro:include filename="$(find agni_description)/calibration/default_cal.xml"/>
+     xmlns:xacro="http://www.ros.org/wiki/xacro">
+  <xacro:include filename="$(find agni_description)/robots/right_kuka_shadow.urdf.xacro" />
+  <xacro:include filename="$(find agni_description)/calibration/default_cal.xml"/>
   <link name="world" />
-  <!-- KUKA arm -->
-  <xacro:kuka_lwr_arm name="right_" reflect="1" tool_name=""/>
-  <joint name="right_frame_placement" type="fixed">
-		<origin xyz="${cal_right_arm_x} ${cal_right_arm_y} ${cal_right_arm_z}"
-				rpy="${cal_right_arm_roll} ${cal_right_arm_pitch} ${cal_right_arm_yaw}"/>
-    <parent link="world"/>
-    <child link="right_arm_base_link"/>
-  </joint>
-  <xacro:right_lwr_arm_gazebo_controller namespace="rk" port="49940"/>
-  <!-- Shadow Hands -->
-  <xacro:shadowhand muscletrans="false" muscle="false" bio="false" ubi="true" eli="false" reflect="1.0" prefix=""  />
-  <xacro:shadow_gazebo_controller_manager namespace="rh" />
-  <!-- Link arm and hand -->
-  <joint name="right_arm_hand_mount" type="fixed">
-    <parent link="right_arm_hand_mount"/>
-    <child link="forearm"/>
-    <origin xyz="0 0 0.0151" rpy="0 0 0" />
-  </joint>
+  <!-- KUKA Shadow arm and hand  -->
+  <xacro:rightkukashadow parent="world" prefix="false" controller="true">
+    <origin xyz="${cal_right_arm_x} ${cal_right_arm_y} ${cal_right_arm_z}"
+        rpy="${cal_right_arm_roll} ${cal_right_arm_pitch} ${cal_right_arm_yaw}"/>
+  </xacro:rightkukashadow>
 </robot>

File: agni_description/robots/right_kuka_shadow_prefix_gazebo.urdf.xacro (robot description, xacro)
@@ -1,28 +1,12 @@
 <?xml version="1.0"?>
 <robot name="right_kuka_shadow"
-		 xmlns:xacro="http://www.ros.org/wiki/xacro">
-  <xacro:include filename="$(find agni_description)/kuka/lwr.urdf.xacro"/>
-  <xacro:include filename="$(find agni_description)/kuka/lwr_controllers.gazebo.xacro"/>
-  <xacro:include filename="$(find agni_description)/urdf/sr_gazebo.urdf.xacro" />
-  <xacro:include filename="$(find sr_description)/hand/xacro/full_hand.urdf.xacro" />
-   <xacro:include filename="$(find agni_description)/calibration/default_cal.xml"/>
+     xmlns:xacro="http://www.ros.org/wiki/xacro">
+  <xacro:include filename="$(find agni_description)/robots/right_kuka_shadow.urdf.xacro" />
+  <xacro:include filename="$(find agni_description)/calibration/default_cal.xml"/>
   <link name="world" />
-  <!-- KUKA arm -->
-  <xacro:kuka_lwr_arm name="right_" reflect="1" tool_name=""/>
-  <joint name="right_frame_placement" type="fixed">
-		<origin xyz="${cal_right_arm_x} ${cal_right_arm_y} ${cal_right_arm_z}"
-				rpy="${cal_right_arm_roll} ${cal_right_arm_pitch} ${cal_right_arm_yaw}"/>
-    <parent link="world"/>
-    <child link="right_arm_base_link"/>
-  </joint>
-  <xacro:right_lwr_arm_gazebo_controller namespace="rk" port="49940"/>
-  <!-- Shadow Hands -->
-  <xacro:shadowhand muscletrans="false" muscle="false" bio="false" ubi="true" eli="false" reflect="1.0" prefix="r_"  />
-  <xacro:shadow_gazebo_controller_manager namespace="rh" />
-  <!-- Link arm and hand -->
-  <joint name="right_arm_hand_mount" type="fixed">
-    <parent link="right_arm_hand_mount"/>
-    <child link="r_forearm"/>
-    <origin xyz="0 0 0.0151" rpy="0 0 0" />
-  </joint>
+  <!-- KUKA Shadow arm and hand  -->
+  <xacro:rightkukashadow parent="world" prefix="true" controller="true">
+    <origin xyz="${cal_right_arm_x} ${cal_right_arm_y} ${cal_right_arm_z}"
+        rpy="${cal_right_arm_roll} ${cal_right_arm_pitch} ${cal_right_arm_yaw}"/>
+  </xacro:rightkukashadow>
 </robot>

File: agni_description/urdf/frame-half.urdf.xacro (robot description, xacro)
@@ -6,66 +6,114 @@
 <xacro:include filename="$(find agni_description)/urdf/util.urdf.xacro"/>
 <xacro:include filename="$(find agni_description)/urdf/materials.urdf.xacro"/>
+<xacro:include filename="$(find agni_description)/calibration/default_cal.xml"/>
+  <property name="cos30"     value="0.866025404" />
+  <property name="sin30"     value="0.5" />
+  <property name="sin60"     value="0.866025404" />
+  <property name="mount_triangle_length"     value="0.26" />
 <xacro:macro name="bar" params="thickness len *origin">
-	 <visual>
-		<xacro:insert_block name="origin"/>
-		<geometry><box size="${thickness} ${thickness} ${len}"/></geometry>
-		<material name="Silver"/>
-	 </visual>
+   <visual>
+    <xacro:insert_block name="origin"/>
+    <geometry><box size="${thickness} ${thickness} ${len}"/></geometry>
+    <material name="Silver"/>
+   </visual>
+   <collision>
+    <xacro:insert_block name="origin"/>
+    <geometry><box size="${thickness} ${thickness} ${len}"/></geometry>
+   </collision>
 </xacro:macro>
 <xacro:macro name="frame-half" params="prefix thickness width depth height tableHeight">
   <link name="${prefix}_frame">
-	 <!-- horizontal front bar-->
-	 <xacro:bar thickness="${thickness}" len="${width}">
-		<origin xyz="0 ${thickness/2} ${-thickness/2}" rpy="0 ${-M_PI/2} 0"/>
-	 </xacro:bar>
-	 <!-- horizontal rear bar -->
-	 <xacro:bar thickness="${thickness}" len="${width}">
-		<origin xyz="0 ${depth+thickness/2} ${-thickness/2}" rpy="0 ${-M_PI/2} 0"/>
-	 </xacro:bar>
-	 <!-- horizontal rear bar top -->
-	 <xacro:bar thickness="${thickness}" len="${width}">
-		<origin xyz="0 ${depth+thickness/2} ${height+thickness/2}" rpy="0 ${-M_PI/2} 0"/>
-	 </xacro:bar>
-	 <!-- left front pole -->
-	 <xacro:bar thickness="${thickness}" len="${thickness+tableHeight}">
-		<origin xyz="${-(width+thickness)/2} ${thickness/2} ${-(thickness+tableHeight)/2}"/>
-	 </xacro:bar>
-	 <!-- right front pole -->
-	 <xacro:bar thickness="${thickness}" len="${thickness+tableHeight}">
-		<origin xyz="${+(width+thickness)/2} ${thickness/2} ${-(thickness+tableHeight)/2}"/>
-	 </xacro:bar>
-	 <!-- left rear pole -->
-	 <xacro:bar thickness="${thickness}" len="${height+2*thickness+tableHeight}">
-		<origin xyz="${-(width+thickness)/2} ${depth+thickness/2} ${(height-tableHeight)/2}"/>
-	 </xacro:bar>
-	 <!-- right rear pole -->
-	 <xacro:bar thickness="${thickness}" len="${height+2*thickness+tableHeight}">
-		<origin xyz="${+(width+thickness)/2} ${depth+thickness/2} ${(height-tableHeight)/2}"/>
-	 </xacro:bar>
-	 <!-- left side bottom -->
-	 <xacro:bar thickness="${thickness}" len="${depth}">
-		<origin xyz="${-(width+thickness)/2} ${depth/2} ${-thickness/2}"
-				  rpy="${-M_PI/2} 0 0"/>
-	 </xacro:bar>
-	 <!-- right side bottom -->
-	 <xacro:bar thickness="${thickness}" len="${depth}">
-		<origin xyz="${+(width+thickness)/2} ${depth/2} ${-thickness/2}"
-				  rpy="${-M_PI/2} 0 0"/>
-	 </xacro:bar>
-	 <!-- left central pole -->
-	 <xacro:bar thickness="${thickness}" len="${thickness+tableHeight+(height)/2}">
-		<origin xyz="${-thickness} ${(depth)/2+2*thickness} ${-(2*tableHeight-height)/4-thickness/2}"/>
-	 </xacro:bar>
-	 <!-- right central pole -->
-	 <xacro:bar thickness="${thickness}" len="${thickness+tableHeight+(height)/2}">
-		<origin xyz="${thickness} ${(depth)/2+2*thickness} ${-(2*tableHeight-height)/4-thickness/2}"/>
-	 </xacro:bar>
-	<!-- table plane -->
-	 <visual>
-	  <origin xyz="0 ${depth/2} -0.01"
-				  rpy="0 0 0"/>
-		<geometry><box size="${width} ${depth} ${0.02}"/></geometry>
-		<material name="Silver"/>
-	 </visual>
+   <!-- horizontal front bar-->
+   <xacro:bar thickness="${thickness}" len="${width}">
+    <origin xyz="0 ${thickness/2} ${-thickness/2}" rpy="0 ${-M_PI/2} 0"/>
+   </xacro:bar>
+   <!-- horizontal rear bar -->
+   <xacro:bar thickness="${thickness}" len="${width}">
+    <origin xyz="0 ${depth+thickness/2} ${-thickness/2}" rpy="0 ${-M_PI/2} 0"/>
+   </xacro:bar>
+   <!-- horizontal rear bar top -->
+   <xacro:bar thickness="${thickness}" len="${width}">
+    <origin xyz="0 ${depth+thickness/2} ${height+thickness/2}" rpy="0 ${-M_PI/2} 0"/>
+   </xacro:bar>
+   <!-- left front pole -->
+   <xacro:bar thickness="${thickness}" len="${thickness+tableHeight}">
+    <origin xyz="${-(width+thickness)/2} ${thickness/2} ${-(thickness+tableHeight)/2}"/>
+   </xacro:bar>
+   <!-- right front pole -->
+   <xacro:bar thickness="${thickness}" len="${thickness+tableHeight}">
+    <origin xyz="${+(width+thickness)/2} ${thickness/2} ${-(thickness+tableHeight)/2}"/>
+   </xacro:bar>
+   <!-- left rear pole -->
+   <xacro:bar thickness="${thickness}" len="${height+2*thickness+tableHeight}">
+    <origin xyz="${-(width+thickness)/2} ${depth+thickness/2} ${(height-tableHeight)/2}"/>
+   </xacro:bar>
+   <!-- right rear pole -->
+   <xacro:bar thickness="${thickness}" len="${height+2*thickness+tableHeight}">
+    <origin xyz="${+(width+thickness)/2} ${depth+thickness/2} ${(height-tableHeight)/2}"/>
+   </xacro:bar>
+   <!-- left side bottom -->
+   <xacro:bar thickness="${thickness}" len="${depth}">
+    <origin xyz="${-(width+thickness)/2} ${depth/2} ${-thickness/2}"
+          rpy="${-M_PI/2} 0 0"/>
+   </xacro:bar>
+   <!-- right side bottom -->
+   <xacro:bar thickness="${thickness}" len="${depth}">
+    <origin xyz="${+(width+thickness)/2} ${depth/2} ${-thickness/2}"
+          rpy="${-M_PI/2} 0 0"/>
+   </xacro:bar>
+   <!-- left central pole -->
+   <xacro:bar thickness="${thickness}" len="${thickness+tableHeight+(height)/2}">
+    <origin xyz="${-thickness} ${(depth)/2+2*thickness} ${-(2*tableHeight-height)/4-thickness/2}"/>
+   </xacro:bar>
+   <!-- right central pole -->
+   <xacro:bar thickness="${thickness}" len="${thickness+tableHeight+(height)/2}">
+    <origin xyz="${thickness} ${(depth)/2+2*thickness} ${-(2*tableHeight-height)/4-thickness/2}"/>
+   </xacro:bar>
+  <!-- kuka mount triangle -->
+   <visual>
+     <origin xyz="${cal_left_arm_x-cos30*0.01} ${cal_left_arm_y} ${cal_left_arm_z-sin30*0.01}"
+        rpy="0 ${M_PI/3} 0"/>
+    <geometry><box size="${mount_triangle_length} ${mount_triangle_length} ${0.02}"/></geometry>
+    <material name="Silver"/>
+   </visual>
+   <collision>
+     <origin xyz="${cal_left_arm_x-cos30*0.01} ${cal_left_arm_y} ${cal_left_arm_z-sin30*0.01}"
+        rpy="0 ${M_PI/3} 0"/>
+    <geometry><box size="${mount_triangle_length} ${mount_triangle_length} ${0.02}"/></geometry>
+   </collision>
+   <visual>
+     <origin xyz="${cal_right_arm_x+cos30*0.01} ${cal_right_arm_y} ${cal_right_arm_z-sin30*0.01}"
+        rpy="0 ${-M_PI/3} 0"/>
+    <geometry><box size="${mount_triangle_length} ${mount_triangle_length} ${0.02}"/></geometry>
+    <material name="Silver"/>
+   </visual>
+    <collision>
+       <origin xyz="${cal_right_arm_x+cos30*0.01} ${cal_right_arm_y} ${cal_right_arm_z-sin30*0.01}"
+        rpy="0 ${-M_PI/3} 0"/>
+    <geometry><box size="${mount_triangle_length} ${mount_triangle_length} ${0.02}"/></geometry>
+   </collision>
+   <visual>
+     <origin xyz="0 ${cal_right_arm_y} ${cal_right_arm_z-sin30*0.02-mount_triangle_length/2*sin60-0.01}"
+        rpy="0 0 0"/>
+    <geometry><box size="${mount_triangle_length} ${mount_triangle_length} ${0.02}"/></geometry>
+    <material name="Silver"/>
+   </visual>
+   <collision>
+      <origin xyz="0 ${cal_right_arm_y} ${cal_right_arm_z-sin30*0.02-mount_triangle_length/2*sin60-0.01}"
+        rpy="0 0 0"/>
+    <geometry><box size="${mount_triangle_length} ${mount_triangle_length} ${0.02}"/></geometry>
+   </collision>
+  <!-- table plane -->
+   <visual>
+    <origin xyz="0 ${depth/2} -0.01"
+          rpy="0 0 0"/>
+    <geometry><box size="${width} ${depth} ${0.02}"/></geometry>
+    <material name="Silver"/>
+   </visual>
+   <collision>
+      <origin xyz="0 ${depth/2} -0.01"
+          rpy="0 0 0"/>
+      <geometry><box size="${width} ${depth} ${0.02}"/></geometry>
+    </collision>
   </link>
   <gazebo reference="${prefix}_frame">
