Commit message: Fixed flobi collision and mesh material, changed kuka meshes to use Y_UP, added monitors in the kuka frame

File: agni_description/flobi/flobi-eye.urdf.xacro (robot description, xacro)
@@ -46,15 +46,9 @@
         <origin xyz="0 0 0" rpy="0 0 0"/>
         <geometry>
-          <mesh scale="1.0 1.0 1.0"
+          <mesh scale="0.1 0.1 0.1"
 					 filename="package://agni_description/flobi/flobi-eye-ball.dae"/>
         </geometry>
         <material name="Orange"/>
       </visual>
-      <collision>
-        <origin xyz="0 0 0" rpy="0 0 0"/>
-        <geometry name="${prefix}flobi_eye_${name}_collision_geom">
-          <box size="0.02 0.02 0.02" />
-        </geometry>
-      </collision>
     </link>
   </macro>

File: agni_description/flobi/flobiv3.urdf.xacro (robot description, xacro)
@@ -26,16 +26,16 @@
         <origin xyz="0 0 0.038" rpy="0 0 0"/>
         <geometry>
-          <mesh scale="1.0 1.0 1.0"
+          <mesh scale="0.1 0.1 0.1"
 					 filename="package://agni_description/flobi/flobi-neck.dae"/>
         </geometry>
-        <material name="Orange"/>
       </visual>
       <collision>
-        <origin xyz="0 0 0" rpy="0 0 0"/>
+        <origin xyz="0 0 0.1" rpy="0 0 0"/>
         <geometry name="${prefix}flobi_neck_collision_geom">
-          <box size="0.05 0.02 0.07" />
+					<cylinder length="0.1" radius="0.07"/>
         </geometry>
       </collision>
     </link>
+     -->
     <joint name="${prefix}floby_neck_pan_joint" type="revolute">
       <origin xyz="0 0 0.0" rpy="0 0 0"/>
@@ -91,13 +91,12 @@
         <origin xyz="0 0 0.008" rpy="0 0 0"/>
         <geometry>
-          <mesh scale="1.0 1.0 1.0"
+          <mesh scale="0.1 0.1 0.1"
 					 filename="package://agni_description/flobi/flobi-head.dae"/>
         </geometry>
-        <material name="Orange"/>
       </visual>
       <collision>
-        <origin xyz="0 0 0" rpy="0 0 0"/>
+        <origin xyz="0 0 0.08" rpy="0 0 0"/>
         <geometry name="${prefix}flobi_head_collision_geom">
-          <box size="0.08 0.08 0.16" />
+          <sphere radius="0.1" />
         </geometry>
       </collision>

File: agni_description/urdf/frame-half.urdf.xacro (robot description, xacro)
@@ -70,4 +70,24 @@
     <origin xyz="${thickness} ${(depth)/2+2*thickness} ${-(2*tableHeight-height)/4-thickness/2}"/>
    </xacro:bar>
+   <!-- virtual protection plane for the screens -->
+    <!-- right screen -->
+   <visual>
+    <origin xyz="${-width/2+0.3} ${depth-thickness} ${height}"
+          rpy="0 0 0"/>
+    <geometry><box size="${0.6} ${0.1} ${0.4}"/></geometry>
+    <material name="Silver"/>
+   </visual>
+    <!-- left screen -->
+   <visual>
+     <origin xyz="${width/2-0.3} ${depth-thickness} ${height}"
+          rpy="0 0 0"/>
+    <geometry><box size="${0.6} ${0.1} ${0.4}"/></geometry>
+    <material name="Silver"/>
+   </visual>
+   <collision>
+      <origin xyz="0 ${depth-2*thickness} ${height/2}"
+          rpy="0 0 0"/>
+      <geometry><box size="${width+2*thickness} ${0.01} ${height+0.4+2*thickness}"/></geometry>
+    </collision>
   <!-- kuka mount triangle -->
    <visual>
